File: mfosish_ww_supply/mfosish_ww_supply.kicad_pcb (KiCad board)
At the start: 2 copper layers, 100 x 61 mm, 31 parts, among them J1 Conn_01x02, J2 Conn_01x03, J3 Conn_01x02, U1 LM7812_TO220, U2 LM7912_TO220

Commit message: Modifications for DIY etching, only one AC connector and 3.81mm pitch connectors.
Parts:
- removed J3: Conn_01x02, ao_tht:TerminalBlock_dinkle_pluggable_2_P5.00mm
- J1: footprint ao_tht:TerminalBlock_dinkle_pluggable_2_P5.00mm -> TerminalBlock_MetzConnect:TerminalBlock_MetzConnect_Type086_RT03402HBLC_1x02_P3.81mm_Horizontal
- J2: footprint ao_tht:TerminalBlock_Degson_DG301_1x03_P5.00mm_Vertical -> TerminalBlock_MetzConnect:TerminalBlock_MetzConnect_Type086_RT03403HBLC_1x03_P3.81mm_Horizontal
- moved J1 31.3 mm to (54.5, 92.5)
- moved D1 15.6 mm to (69.0, 66.5), turned to 180 degrees
- moved C7 11.0 mm to (111.0, 88.0)
- moved C1 10.9 mm to (63.0, 75.1)
- moved C3 10.9 mm to (83.0, 75.1)
- moved C5 10.9 mm to (103.0, 75.1)
- moved J2 4.01 mm to (145.5, 91.0)
Routing:
- net Net-(D1-Pad2): track 88.8 -> 59.2 mm
- net Net-(C1-Pad1): track 78.7 -> 88.1 mm
- net Net-(C2-Pad2): track 101.9 -> 105.0 mm
- net Net-(C9-Pad1): track 55.6 -> 57.4 mm
- net -12V: track 14.8 -> 16.1 mm
- net +12V: track 14.3 -> 15.5 mm
Other:
- net class PWR added: clearance 0.2, trace_width 2, via_dia 0.8, via_drill 0.4

Commit message: Few more cleanups
Repositioned D1/D2,  Cleaned up labels, redid a few wonky traces
Parts:
- moved D1 26.3 mm to (62.5, 92.0), turned to 0 degrees
- moved D2 25.9 mm to (62.5, 97.0)
Routing:
- net Net-(D1-Pad2): track 59.2 -> 20.5 mm
- net Net-(C2-Pad2): track 105.0 -> 115.3 mm
- net Net-(C1-Pad1): track 88.1 -> 96.2 mm
- net Net-(C9-Pad1): track 57.4 -> 56.8 mm
